Commit message: Fixed urdf file references to work on linux

File: src/sim/roman.urdf (robot description, URDF)
Before this commit: robot roman, 24 links, 23 joints
Links:
- link finger_1_link_0: geometry collision mesh filename=package://meshes/robotiq-3f-gripper/collision/link_0.STL; visual mesh filename=package://meshes/robotiq-3f-gripper/visual/link_0.dae
- link finger_1_link_1: geometry collision mesh filename=package://meshes/robotiq-3f-gripper/collision/link_1.STL; visual mesh filename=package://meshes/robotiq-3f-gripper/visual/link_1.dae
- link finger_1_link_2: geometry collision mesh filename=package://meshes/robotiq-3f-gripper/collision/link_2.STL; visual mesh filename=package://meshes/robotiq-3f-gripper/visual/link_2.dae
- link finger_1_link_3: geometry collision mesh filename=package://meshes/robotiq-3f-gripper/collision/link_3.STL; visual mesh filename=package://meshes/robotiq-3f-gripper/visual/link_3.dae
- link finger_2_link_0: geometry collision mesh filename=package://meshes/robotiq-3f-gripper/collision/link_0.STL; visual mesh filename=package://meshes/robotiq-3f-gripper/visual/link_0.dae
- link finger_2_link_1: geometry collision mesh filename=package://meshes/robotiq-3f-gripper/collision/link_1.STL; visual mesh filename=package://meshes/robotiq-3f-gripper/visual/link_1.dae
- link finger_2_link_2: geometry collision mesh filename=package://meshes/robotiq-3f-gripper/collision/link_2.STL; visual mesh filename=package://meshes/robotiq-3f-gripper/visual/link_2.dae
- link finger_2_link_3: geometry collision mesh filename=package://meshes/robotiq-3f-gripper/collision/link_3.STL; visual mesh filename=package://meshes/robotiq-3f-gripper/visual/link_3.dae
- link finger_middle_link_0: geometry collision mesh filename=package://meshes/robotiq-3f-gripper/collision/link_0.STL; visual mesh filename=package://meshes/robotiq-3f-gripper/visual/link_0.dae
- link finger_middle_link_1: geometry collision mesh filename=package://meshes/robotiq-3f-gripper/collision/link_1.STL; visual mesh filename=package://meshes/robotiq-3f-gripper/visual/link_1.dae
- link finger_middle_link_2: geometry collision mesh filename=package://meshes/robotiq-3f-gripper/collision/link_2.STL; visual mesh filename=package://meshes/robotiq-3f-gripper/visual/link_2.dae
- link finger_middle_link_3: geometry collision mesh filename=package://meshes/robotiq-3f-gripper/collision/link_3.STL; visual mesh filename=package://meshes/robotiq-3f-gripper/visual/link_3.dae
- link palm: geometry collision mesh filename=package://meshes/robotiq-3f-gripper/collision/palm.STL; visual mesh filename=package://meshes/robotiq-3f-gripper/visual/palm.dae

Commit message: combined arm and sim code paths

File: src/sim/roman.urdf (robot description, URDF)
Before this commit: robot roman, 24 links, 23 joints
Links:
- added link tcp_link, mass 0; collision box size=0.01 0.01 0.01
Joints:
- added joint tcp_fixed_joint: type fixed, parent wrist_3_link, child tcp_link, origin xyz=0.0 0.215 0.0 rpy=0.0 0.0 1.57079632679
- joint gripper_fixed_joint: origin xyz=0.0 0.0575 0.0 rpy=0.0 0.0 0.0 -> xyz=0.0 0.0575 0.0 rpy=0.0 3.1415 0.0
