Commit message: various fixes in sim to match the real robot

File: src/roman/sim/ur_rq3.urdf (robot description, URDF)
Before this commit: robot roman, 25 links, 24 joints
Links:
- removed link tcp_link
- added link grasp_point; collision box size=0.01 0.01 0.01
- added link gripper_mount, mass 0.1; collision cylinder length=0.0275 radius=0.0375; visual cylinder length=0.0275 radius=0.0375
Joints:
- removed joint tcp_fixed_joint
- added joint gripper_fixed_mount_joint: type fixed, parent ft_sensor, child gripper_mount, origin xyz=0.0 0.034 0.0 rpy=0.0 0.0 0.0
- added joint tool0-grasp_point_fixed_joint: type fixed, parent tool0, child grasp_point, origin xyz=0.0 0.0 0.260 rpy=0.0 0.0 0.0
- joint ft_sensor_fixed_joint: origin xyz=0.0 0.1 0.0 rpy=0.0 0.0 0.0 -> xyz=0.0 0.101 0.0 rpy=0.0 0.0 0.0
- joint gripper_fixed_joint: origin xyz=0.0 0.0575 0.0 rpy=0.0 3.1415 0.0 -> xyz=0.0 0.0475 0.0 rpy=0.0 3.1415 0.0; parent ft_sensor -> gripper_mount

Commit message: fixed force-based contact detection cleaned up tests

File: src/roman/sim/ur_rq3.urdf (robot description, URDF)
Before this commit: robot roman, 26 links, 25 joints
Links:
- link grasp_point: geometry visual box size=0.01 0.01 0.01

Commit message: cleanup

File: src/roman/sim/ur_rq3.urdf (robot description, URDF)
Before this commit: robot roman, 26 links, 25 joints
Links:
- link grasp_point: mass None -> 0.0
- link tool0: mass None -> 0.0

Commit message: Sim improvements: 1. Added sim support for Robotiq 3F Gripper 2. Added sim support for wrist FT sensor 3. Added mechanism for configuring the sim scene

File: src/roman/sim/ur_rq3.urdf (robot description, URDF)
Before this commit: robot roman, 26 links, 25 joints
Joints:
- joint finger_1_joint_2: limit lower=0 upper=3.1416 effort=100 velocity=100 -> lower=-1 upper=1 effort=100 velocity=100
- joint finger_1_joint_3: limit lower=0 upper=3.1416 effort=100 velocity=100 -> lower=-1 upper=1 effort=100 velocity=100
- joint finger_2_joint_2: limit lower=0 upper=3.1416 effort=100 velocity=100 -> lower=-1 upper=1 effort=100 velocity=100
- joint finger_2_joint_3: limit lower=0 upper=3.1416 effort=100 velocity=100 -> lower=-1 upper=1 effort=100 velocity=100
- joint finger_middle_joint_2: limit lower=0 upper=3.1416 effort=100 velocity=100 -> lower=-1 upper=1 effort=100 velocity=100
- joint finger_middle_joint_3: limit lower=0 upper=3.1416 effort=100 velocity=100 -> lower=-1 upper=1 effort=100 velocity=100
- joint ft_sensor_fixed_joint: origin xyz=0.0 0.101 0.0 rpy=0.0 0.0 0.0 -> xyz=0.0 0.101 0.0 rpy=-1.570796326 0  0
- joint gripper_fixed_joint: origin xyz=0.0 0.0475 0.0 rpy=0.0 3.1415 0.0 -> xyz=0.0  0.0 0.0475 rpy=-1.570796326 3.1415 0.0
- joint gripper_fixed_mount_joint: origin xyz=0.0 0.034 0.0 rpy=0.0 0.0 0.0 -> xyz=0.0 0.0 0.034 rpy=0.0 0.0 0.0

Commit message: Added sim support for pinch grasp

File: src/roman/sim/ur_rq3.urdf (robot description, URDF)
Before this commit: robot roman, 26 links, 25 joints
Links:
- link finger_1_link_0: geometry visual mesh filename=package://meshes/robotiq-3f-gripper/visual/link_0.dae
- link finger_2_link_0: geometry visual mesh filename=package://meshes/robotiq-3f-gripper/visual/link_0.dae
