Commit message: adjustments to match hardware install

File: roman/sim/ur_rq3.urdf (robot description, URDF)
Before this commit: robot roman, 26 links, 25 joints
Joints:
- joint gripper_fixed_mount_joint: origin xyz=0.0 0.0 0.034 rpy=0.0 0.0 0.0 -> xyz=0.0 0.0 0.034 rpy=0.0 0.0 0.262
- joint wrist_3_link-tool0_fixed_joint: origin xyz=0 0.0823 0 rpy=-1.570796325 0 0 -> xyz=0 0.0623 0 rpy=-1.570796325 0 0

Commit message: sim: removed tooltip marker

File: roman/sim/ur_rq3.urdf (robot description, URDF)
Before this commit: robot roman, 26 links, 25 joints
Links:
- link grasp_point: mass 0.0 -> None; geometry 
